Commit message: Cambios en el archivo URDF

File: src/rona_robot/description/robot_core.xacro (robot description, xacro)
@@ -3,10 +3,10 @@
     <xacro:include filename="inertial_macros.xacro"/>
     <!--medidas del chasis-->
-    <xacro:property name="chassis_length" value="0.335"/>
-    <xacro:property name="chassis_width" value="0.265"/>
-    <xacro:property name="chassis_height" value="0.138"/>
+    <xacro:property name="chassis_length" value="0.400"/>
+    <xacro:property name="chassis_width" value="0.1"/>
+    <xacro:property name="chassis_height" value="0.15"/>
     <xacro:property name="chassis_mass" value="1.0"/>
-    <xacro:property name="wheel_radius" value="0.033"/>
-    <xacro:property name="wheel_thickness" value="0.026"/>
+    <xacro:property name="wheel_radius" value="0.05"/>
+    <xacro:property name="wheel_thickness" value="0.01"/>
     <xacro:property name="wheel_mass" value="0.05"/>
     <xacro:property name="wheel_offset_x" value="0.226"/>
@@ -59,5 +59,5 @@
                 <box size="${chassis_length} ${chassis_width} ${chassis_height}"/>
             </geometry>
-            <material name="orange"/>
+            <material name="blue"/>
         </visual>
         <collision>
@@ -74,5 +74,5 @@
         <material>Gazebo/Orange</material>
     </gazebo>
-    <!-- LEFT WHEEL LINK -->
+    <!-- FRONT LEFT WHEEL LINK -->
     <!-- Podríamos conectarlo al chasis. Pero en este caso se conecta a la base porque su origen es el centro de rotación de las ruedas-->
     <joint name="left_wheel_joint" type="continuous">
@@ -83,5 +83,5 @@
         <origin xyz="0 ${wheel_offset_y} 0" rpy="-${pi/2} 0 0" />
         <!-- Especificamos un eje de rotacion. Nos tenemos que preguntar -->
-        <!-- ¿Cuando la rueda tiene un movimiento positivo, en qué dirección está girando? En este caso es positivo alrededor de Z-->
+        <!-- Cuando la rueda tiene un movimiento positivo, ¿en qué dirección está girando? En este caso es positivo alrededor de Z-->
         <axis xyz="0 0 1"/>
     </joint>
@@ -89,7 +89,7 @@
         <visual>
             <geometry>
-                <cylinder radius="${wheel_radius}" length="${wheel_thickness}"/>
-            </geometry>
-            <material name="blue"/>
+                <cylinder radius="0,05" length="0,1"/>
+            </geometry>
+            <material name="orange"/>
         </visual>
         <collision>
@@ -105,5 +105,5 @@
         <material>Gazebo/Blue</material>
     </gazebo>
-    <!-- RIGHT WHEEL LINK -->
+    <!-- FRONT RIGHT WHEEL LINK -->
     <joint name="right_wheel_joint" type="continuous">
         <parent link="base_link"/>
@@ -115,5 +115,57 @@
         <visual>
             <geometry>
-                <cylinder radius="${wheel_radius}" length="${wheel_thickness}"/>
+                <cylinder radius="0,05" length="0,1"/>
+            </geometry>
+            <material name="blue"/>
+        </visual>
+        <collision>
+            <geometry>
+                <sphere radius="${wheel_radius}"/>
+            </geometry>
+        </collision>
+        <xacro:inertial_cylinder mass="${wheel_mass}" length="${wheel_thickness}" radius="${wheel_radius}">
+            <origin xyz="0 0 0" rpy="0 0 0"/>
+        </xacro:inertial_cylinder>
+    </link>
+    <gazebo reference="right_wheel">
+        <material>Gazebo/Blue</material>
+    </gazebo>
+<!-- REAR RIGHT WHEEL LINK -->
+    <joint name="right_wheel_joint" type="continuous">
+        <parent link="base_link"/>
+        <child link="right_wheel"/>
+        <origin xyz="0 ${-wheel_offset_y} 0" rpy="${pi/2} 0 0" />
+        <axis xyz="0 0 -1"/>
+    </joint>
+    <link name="right_wheel">
+        <visual>
+            <geometry>
+                <cylinder radius="0,05" length="0,1"/>
+            </geometry>
+            <material name="blue"/>
+        </visual>
+        <collision>
+            <geometry>
+                <sphere radius="${wheel_radius}"/>
+            </geometry>
+        </collision>
+        <xacro:inertial_cylinder mass="${wheel_mass}" length="${wheel_thickness}" radius="${wheel_radius}">
+            <origin xyz="0 0 0" rpy="0 0 0"/>
+        </xacro:inertial_cylinder>
+    </link>
+    <gazebo reference="right_wheel">
+        <material>Gazebo/Blue</material>
+    </gazebo>
+<!-- REAR RIGHT WHEEL LINK -->
+    <joint name="right_wheel_joint" type="continuous">
+        <parent link="base_link"/>
+        <child link="right_wheel"/>
+        <origin xyz="0 ${-wheel_offset_y} 0" rpy="${pi/2} 0 0" />
+        <axis xyz="0 0 -1"/>
+    </joint>
+    <link name="right_wheel">
+        <visual>
+            <geometry>
+                <cylinder radius="0,05" length="0,1"/>
             </geometry>
             <material name="blue"/>

Commit message: Añadida la macro para crear los rollers de las ruedas omnidireccionales

File: src/rona_robot/description/robot_core.xacro (robot description, xacro)
@@ -2,5 +2,5 @@
 <robot xmlns:xacro="http://www.ros.org/wiki/xacro" >
 <!-- In this file the basic structure of the omnidirectional robot RONA is described -->
-    <!-- MACROS SECTION START-->
+    <!-- MACROS & PROPERTIES SECTION START-->
     <!-- Chassis measures -->
     <xacro:property name="chassis_length" value="0.297"/>
@@ -8,8 +8,46 @@
     <xacro:property name="chassis_height" value="0.09"/>
     <!-- En rviz el eje X es el rojo, el Y el verde y el Z el azul -->
+    <!-- Wheels offsets -->
     <xacro:property name="wheel_offset_y" value="${chassis_width/2 + 0.025}"/>
     <xacro:property name="wheel_offset_x" value="${chassis_length/2 - 0.051}"/>
     <xacro:property name="wheel_offset_z" value="0.028"/>
-    <!-- MACROS SECTION END -->
+    <!-- Rollers measures -->
+    <xacro:property name="roller_diameter" value="0.01"/>
+    <xacro:property name="roller_length" value="0.01"/>
+    <xacro:macro name="roller" params="prefix suffix theta side">
+        <link name="${prefix}_${suffix}_roller">
+            <visual>
+                <origin xyz="0 0 0" rpy="0 ${pi/2} 0" />
+                <geometry>
+                    <cylinder radius="${roller_diameter}" length="${roller_length}"/>
+                </geometry>
+                <material name="black"/>
+            </visual>
+            <collision>
+                <origin xyz="0 0 0" rpy="0 ${pi/2} 0" />
+                <geometry>
+                    <cylinder radius="${roller_diameter}" length="${roller_length}"/>
+                </geometry>
+            </collision>
+            <xacro:roller_inertial mass="0.001"/>
+        </link>
+        <joint name="${prefix}_${suffix}_roller_joint" type="continuous">
+            <axis xyz="1 0 0" />
+            <parent link="${prefix}_wheel"/>
+            <child link="${prefix}_${suffix}_roller"/>
+            <origin xyz="${sin(theta)*roller_radius} ${roller_side_length*side} ${cos(theta)*roller_radius}" rpy="0 ${theta} 0"/>
+            <dynamics damping="0.0001" />
+        </joint>
+        <!-- This block provides the simulator (Gazebo) with information on a few additional
+        physical properties. See http://gazebosim.org/tutorials/?tut=ros_urdf for more-->
+        <gazebo reference="${prefix}_${suffix}_roller">
+            <mu1 value="2000.0"/>
+            <mu2 value="1000.0"/>
+            <kp value="10000000.0" />
+            <kd value="1.0" />
+            <material>Gazebo/Grey</material>
+        </gazebo>
+    </xacro:macro>
+    <!-- MACROS & PROPERTIES SECTION END -->
     <!-- COLOR DESCRIPTIONS START -->
     <material name="white">
@@ -44,5 +82,4 @@
             <geometry>
                 <box size="${chassis_length} ${chassis_width} ${chassis_height}"/>
-                <!-- <box size="0.3 0.3 0.15"/> -->
             </geometry>
             <material name="blue"/>

Commit message: Añadidos los rollers de las ruedas omnidireccionales

File: src/rona_robot/description/robot_core.xacro (robot description, xacro)
@@ -2,52 +2,4 @@
 <robot xmlns:xacro="http://www.ros.org/wiki/xacro" >
 <!-- In this file the basic structure of the omnidirectional robot RONA is described -->
-    <!-- MACROS & PROPERTIES SECTION START-->
-    <!-- Chassis measures -->
-    <xacro:property name="chassis_length" value="0.297"/>
-    <xacro:property name="chassis_width" value="0.188"/>
-    <xacro:property name="chassis_height" value="0.09"/>
-    <!-- En rviz el eje X es el rojo, el Y el verde y el Z el azul -->
-    <!-- Wheels offsets -->
-    <xacro:property name="wheel_offset_y" value="${chassis_width/2 + 0.025}"/>
-    <xacro:property name="wheel_offset_x" value="${chassis_length/2 - 0.051}"/>
-    <xacro:property name="wheel_offset_z" value="0.028"/>
-    <!-- Rollers measures -->
-    <xacro:property name="roller_diameter" value="0.01"/>
-    <xacro:property name="roller_length" value="0.01"/>
-    <xacro:macro name="roller" params="prefix suffix theta side">
-        <link name="${prefix}_${suffix}_roller">
-            <visual>
-                <origin xyz="0 0 0" rpy="0 ${pi/2} 0" />
-                <geometry>
-                    <cylinder radius="${roller_diameter}" length="${roller_length}"/>
-                </geometry>
-                <material name="black"/>
-            </visual>
-            <collision>
-                <origin xyz="0 0 0" rpy="0 ${pi/2} 0" />
-                <geometry>
-                    <cylinder radius="${roller_diameter}" length="${roller_length}"/>
-                </geometry>
-            </collision>
-            <xacro:roller_inertial mass="0.001"/>
-        </link>
-        <joint name="${prefix}_${suffix}_roller_joint" type="continuous">
-            <axis xyz="1 0 0" />
-            <parent link="${prefix}_wheel"/>
-            <child link="${prefix}_${suffix}_roller"/>
-            <origin xyz="${sin(theta)*roller_radius} ${roller_side_length*side} ${cos(theta)*roller_radius}" rpy="0 ${theta} 0"/>
-            <dynamics damping="0.0001" />
-        </joint>
-        <!-- This block provides the simulator (Gazebo) with information on a few additional
-        physical properties. See http://gazebosim.org/tutorials/?tut=ros_urdf for more-->
-        <gazebo reference="${prefix}_${suffix}_roller">
-            <mu1 value="2000.0"/>
-            <mu2 value="1000.0"/>
-            <kp value="10000000.0" />
-            <kd value="1.0" />
-            <material>Gazebo/Grey</material>
-        </gazebo>
-    </xacro:macro>
-    <!-- MACROS & PROPERTIES SECTION END -->
     <!-- COLOR DESCRIPTIONS START -->
     <material name="white">
@@ -67,8 +19,94 @@
     </material>
     <!-- COLOR DESCRIPTIONS END -->
+    <!-- PROPERTIES SECTION START-->
+    <!-- Chassis measures -->
+    <xacro:property name="chassis_length" value="0.297"/>
+    <xacro:property name="chassis_width" value="0.188"/>
+    <xacro:property name="chassis_height" value="0.09"/>
+    <!-- En rviz el eje X es el rojo, el Y el verde y el Z el azul -->
+    <!-- Wheels parameters -->
+    <xacro:property name="wheel_offset_y" value="${chassis_width/2 + 0.025}"/>
+    <xacro:property name="wheel_offset_x" value="${chassis_length/2 - 0.051}"/>
+    <xacro:property name="wheel_offset_z" value="0.028"/>
+    <xacro:property name="wheel_radius" value="0.0375"/>
+    <!-- Rollers measures -->
+    <xacro:property name="roller_diameter" value="0.01"/>
+    <xacro:property name="roller_length" value="0.01"/>
+    <!-- PROPERTIES SECTION END -->
     <!-- ROBOT DESCRIPTION START -->
     <!-- Base link -->
     <link name="base_link">
     </link>
+    <xacro:macro name="roller" params="prefix suffix theta roller_orientation">
+        <link name="${prefix}_${suffix}_roller">
+            <visual>
+                <origin xyz="0 0 0" rpy="0 0 0" />
+                <geometry>
+                    <cylinder radius="0,0082" length="0,045"/>
+                </geometry>
+                <material name="black"/>
+            </visual>
+            <collision>
+                <origin xyz="0 0 0" rpy="0 ${pi/4} 0" />
+                <geometry>
+                    <cylinder radius="0,01" length="0,032"/>
+                </geometry>
+            </collision>
+            <!-- <xacro:roller_inertial mass="0.001"/> -->
+        </link>
+        <joint name="${prefix}_${suffix}_roller_joint" type="continuous">
+            <axis xyz="1 0 0" />
+            <parent link="${prefix}_wheel"/>
+            <child link="${prefix}_${suffix}_roller"/>
+            <origin xyz="${cos(theta)*wheel_radius} ${sin(theta)*wheel_radius} 0" rpy="0 ${roller_orientation} ${(pi/2)+theta}"/>
+            <dynamics damping="0.0001" />
+        </joint>
+        <!-- This block provides the simulator (Gazebo) with information on a few additional
+        physical properties. See http://gazebosim.org/tutorials/?tut=ros_urdf for more-->
+        <gazebo reference="${prefix}_${suffix}_roller">
+            <mu1 value="2000.0"/>
+            <mu2 value="1000.0"/>
+            <kp value="10000000.0" />
+            <kd value="1.0" />
+            <material>Gazebo/Grey</material>
+        </gazebo>
+    </xacro:macro>
+    <xacro:macro name="wheel" params="prefix suffix radius length mass offset_x offset_y offset_z wheel_roller_orientation">
+        <link name="${prefix}_${suffix}_wheel">
+            <visual>
+                <origin xyz="0 0 0" rpy="0 0 0"/>
+                <geometry>
+                    <cylinder radius="${radius}" length="${length}"/>
+                </geometry>
+                <material name="orange"/>
+            </visual>
+            <collision>
+                <origin xyz="0 0 0" rpy="0 0 0"/>
+                <geometry>
+                    <cylinder radius="${radius}" length="${length}"/>
+                </geometry>
+            </collision>
+            <!-- <xacro:roller_inertial mass="${mass}"/>     -->
+        </link>
+        <joint name="${prefix}_${suffix}_wheel_joint" type="continuous">
+            <parent link="base_link"/>
+            <child link="${prefix}_${suffix}_wheel"/>
+            <origin xyz="${offset_x} ${offset_y} ${offset_z}" rpy="-${pi/2} 0 0"/>
+            <axis xyz="0 0 1"/>
+        </joint>
+        <gazebo reference="front_left_wheel">
+            <material>Gazebo/Orange</material>
+        </gazebo>
+        <xacro:roller prefix="${prefix}_${suffix}" suffix="one" theta="${2*pi*(1/10)}" roller_orientation="${wheel_roller_orientation}"/>
+        <xacro:roller prefix="${prefix}_${suffix}" suffix="two" theta="${2*pi*(2/10)}" roller_orientation="${wheel_roller_orientation}"/>
+        <xacro:roller prefix="${prefix}_${suffix}" suffix="thr" theta="${2*pi*(3/10)}" roller_orientation="${wheel_roller_orientation}"/>
+        <xacro:roller prefix="${prefix}_${suffix}" suffix="for" theta="${2*pi*(4/10)}" roller_orientation="${wheel_roller_orientation}"/>
+        <xacro:roller prefix="${prefix}_${suffix}" suffix="fve" theta="${2*pi*(5/10)}" roller_orientation="${wheel_roller_orientation}"/>
+        <xacro:roller prefix="${prefix}_${suffix}" suffix="six" theta="${2*pi*(6/10)}" roller_orientation="${wheel_roller_orientation}"/>
+        <xacro:roller prefix="${prefix}_${suffix}" suffix="svn" theta="${2*pi*(7/10)}" roller_orientation="${wheel_roller_orientation}"/>
+        <xacro:roller prefix="${prefix}_${suffix}" suffix="ate" theta="${2*pi*(8/10)}" roller_orientation="${wheel_roller_orientation}"/>
+        <xacro:roller prefix="${prefix}_${suffix}" suffix="nne" theta="${2*pi*(9/10)}" roller_orientation="${wheel_roller_orientation}"/>
+        <xacro:roller prefix="${prefix}_${suffix}" suffix="ten" theta="${2*pi*(10/10)}" roller_orientation="${wheel_roller_orientation}"/>
+    </xacro:macro>
     <!-- Chassis -->
     <joint name="chassis_joint" type="fixed">
@@ -96,95 +134,11 @@
     </gazebo>
     <!-- Front left wheel -->
-    <joint name="front_left_wheel_joint" type="continuous">
-        <parent link="base_link"/>
-        <child link="front_left_wheel"/>
-        <origin xyz="${wheel_offset_x} ${wheel_offset_y} ${wheel_offset_z}" rpy="-${pi/2} 0 0"/>
-        <axis xyz="0 0 1"/>
-    </joint>
-    <link name="front_left_wheel">
-        <visual>
-            <geometry>
-                <cylinder radius="0,0375" length="0,05"/>
-            </geometry>
-            <material name="orange"/>
-        </visual>
-        <collision>
-            <geometry>
-                <cylinder radius="0,04" length="0,05"/>
-            </geometry>
-        </collision>
-    </link>
-    <gazebo reference="front_left_wheel">
-        <material>Gazebo/Orange</material>
-    </gazebo>
+    <xacro:wheel prefix="front" suffix="left" radius="0,0375" length="0,05" mass="0.4" offset_x="${wheel_offset_x}" offset_y="${wheel_offset_y}" offset_z="${wheel_offset_z}" wheel_roller_orientation="${pi/4}"/>
     <!-- Front right wheel -->
-    <joint name="front_right_wheel_joint" type="continuous">
-        <parent link="base_link"/>
-        <child link="front_right_wheel"/>
-        <origin xyz="${wheel_offset_x} ${-wheel_offset_y} ${wheel_offset_z}" rpy="-${pi/2} 0 0"/>
-        <axis xyz="0 0 1"/>
-    </joint>
-    <link name="front_right_wheel">
-        <visual>
-            <geometry>
-                <cylinder radius="0,0375" length="0,05"/>
-            </geometry>
-            <material name="orange"/>
-        </visual>
-        <collision>
-            <geometry>
-                <cylinder radius="0,04" length="0,05"/>
-            </geometry>
-        </collision>
-    </link>
-    <gazebo reference="front_right_wheel">
-        <material>Gazebo/Orange</material>
-    </gazebo>
+    <xacro:wheel prefix="front" suffix="right" radius="0,0375" length="0,05" mass="0.4" offset_x="${wheel_offset_x}" offset_y="${-wheel_offset_y}" offset_z="${wheel_offset_z}" wheel_roller_orientation="${-pi/4}"/>
     <!-- Back left wheel -->
-    <joint name="back_left_wheel_joint" type="continuous">
-        <parent link="base_link"/>
-        <child link="back_left_wheel"/>
-        <origin xyz="${-wheel_offset_x} ${wheel_offset_y} ${wheel_offset_z}" rpy="-${pi/2} 0 0"/>
-        <axis xyz="0 0 1"/>
-    </joint>
-    <link name="back_left_wheel">
-        <visual>
-            <geometry>
-                <cylinder radius="0,0375" length="0,05"/>
-            </geometry>
-            <material name="orange"/>
-        </visual>
-        <collision>
-            <geometry>
-                <cylinder radius="0,04" length="0,05"/>
-            </geometry>
-        </collision>
-    </link>
-    <gazebo reference="back_left_wheel">
-        <material>Gazebo/Orange</material>
-    </gazebo>
+    <xacro:wheel prefix="back" suffix="left" radius="0,0375" length="0,05" mass="0.4" offset_x="${-wheel_offset_x}" offset_y="${wheel_offset_y}" offset_z="${wheel_offset_z}" wheel_roller_orientation="${-pi/4}"/>
     <!-- Back right wheel -->
-    <joint name="back_right_wheel_joint" type="continuous">
-        <parent link="base_link"/>
-        <child link="back_right_wheel"/>
-        <origin xyz="${-wheel_offset_x} ${-wheel_offset_y} ${wheel_offset_z}" rpy="-${pi/2} 0 0"/>
-        <axis xyz="0 0 1"/>
-    </joint>
-    <link name="back_right_wheel">
-        <visual>
-            <geometry>
-                <cylinder radius="0,0375" length="0,05"/>
-            </geometry>
-            <material name="orange"/>
-        </visual>
-        <collision>
-            <geometry>
-                <cylinder radius="0,04" length="0,05"/>
-            </geometry>
-        </collision>
-    </link>
-    <gazebo reference="back_right_wheel">
-        <material>Gazebo/Orange</material>
-    </gazebo>
+    <xacro:wheel prefix="back" suffix="right" radius="0,0375" length="0,05" mass="0.4" offset_x="${-wheel_offset_x}" offset_y="${-wheel_offset_y}" offset_z="${wheel_offset_z}" wheel_roller_orientation="${pi/4}"/>
    <!-- ROBOT DESCRIPTION END -->
 </robot>

Commit message: Ahora el robot no está dentro del suelo

File: src/rona_robot/description/robot_core.xacro (robot description, xacro)
@@ -48,7 +48,7 @@
             </visual>
             <collision>
-                <origin xyz="0 0 0" rpy="0 ${pi/4} 0" />
+                <origin xyz="0 0 0" rpy="0 0 0" />
                 <geometry>
-                    <cylinder radius="0,01" length="0,032"/>
+                    <cylinder radius="0,0082" length="0,045"/>
                 </geometry>
             </collision>
@@ -90,5 +90,5 @@
         </link>
         <joint name="${prefix}_${suffix}_wheel_joint" type="continuous">
-            <parent link="base_link"/>
+            <parent link="chassis"/>
             <child link="${prefix}_${suffix}_wheel"/>
             <origin xyz="${offset_x} ${offset_y} ${offset_z}" rpy="-${pi/2} 0 0"/>
@@ -113,5 +113,5 @@
         <parent link="base_link"/>
         <child link="chassis"/>
-        <origin xyz="0 0 0"/>
+        <origin xyz="0 0 0.022"/>
     </joint>
     <link name="chassis">

Commit message: Cambio del eje de rotacion de los roller

File: src/rona_robot/description/robot_core.xacro (robot description, xacro)
@@ -2,4 +2,5 @@
 <robot xmlns:xacro="http://www.ros.org/wiki/xacro" >
 <!-- In this file the basic structure of the omnidirectional robot RONA is described -->
+    <xacro:include filename="inertial_macros.xacro"/>
     <!-- COLOR DESCRIPTIONS START -->
     <material name="white">
@@ -53,8 +54,10 @@
                 </geometry>
             </collision>
-            <!-- <xacro:roller_inertial mass="0.001"/> -->
+            <xacro:inertial_cylinder mass="0.001" length="0.045" radius="0.0082">
+                <origen xyz="0 0 0" rpy="0 0 0"/>
+            </xacro:inertial_cylinder>
         </link>
         <joint name="${prefix}_${suffix}_roller_joint" type="continuous">
-            <axis xyz="1 0 0" />
+            <axis xyz="0 0 1" />
             <parent link="${prefix}_wheel"/>
             <child link="${prefix}_${suffix}_roller"/>
@@ -129,4 +132,7 @@
             </geometry>
         </colission>
+        <xacro:inertial_box mass="3" x="${chassis_length}" y="${chassis_width}" z="${chassis_height}">
+            <origin xyz="0 0 ${chassis_length}" rpy="0 0 0"/>
+        </xacro:inertial_box>
     </link>
     <gazebo reference="chassis">
