Commit message: .gitignore added and src files modified

File: src/rona_robot/description/macros.xacro (robot description, xacro)
@@ -2,4 +2,5 @@
 <robot xmlns:xacro="http://www.ros.org/wiki/xacro" >
     <xacro:include filename="physical_properties.xacro"/>
+    <xacro:include filename="inertial_macros.xacro"/>
     <xacro:macro name="roller" params="prefix suffix theta roller_orientation">
         <link name="${prefix}_${suffix}_roller">

File: src/rona_robot/description/robot.urdf.xacro (robot description, xacro)
@@ -3,5 +3,5 @@
     <xacro:arg name="use_ros2_control" default="true"/>
     <xacro:arg name="sim_mode" default="false"/>
-    <xacro:include filename="robot_core.xacro" />
+    <xacro:include filename="robot_core_prueba.xacro" />
     <xacro:if value="$(arg use_ros2_control)">
         <xacro:include filename="ros2_control.xacro" />

File: src/rona_robot/description/robot_core.xacro (robot description, xacro)
@@ -47,6 +47,3 @@
     <xacro:wheel prefix="back" suffix="right" radius="0,0375" length="0,05" mass="0.4" offset_x="${-wheel_offset_x}" offset_y="${-wheel_offset_y}" offset_z="${wheel_offset_z}" wheel_roller_orientation="${pi/4}"/>
     <!-- ROBOT DESCRIPTION END -->
-    <gazebo reference="front_left_wheel">
-        <material>Gazebo/Orange</material>
-    </gazebo>
 </robot>
