Commit message: need different approach

File: src/rona_robot/robot_description/physical_properties.xacro (robot description, xacro)
@@ -12,5 +12,5 @@
     <xacro:property name="wheel_radius" value="0.0375"/>
     <!-- Rollers measures -->
-    <xacro:property name="roller_diameter" value="0,01"/>
-    <xacro:property name="roller_length" value="0,01"/>
+    <xacro:property name="roller_diameter" value="0.01"/>
+    <xacro:property name="roller_length" value="0.01"/>
 </robot>

File: src/rona_robot/robot_description/roller.xacro (robot description, xacro)
@@ -5,5 +5,5 @@
         <link name="${prefix}_${suffix}_roller">
             <visual>
-                <origin xyz="0 0 0" rpy="0 0 0" />
+                <origin xyz="-0.5 -0.5 0" rpy="0 0 0" />
                 <geometry>
                     <mesh scale="0.001 0.001 0.001" filename="package://rona_robot/meshes/MecanumWheel_Roller.stl" />
