Commit message: now wheels are shown correctly

File: src/rona_robot/robot_description/front_right_wheel.xacro (robot description, xacro)
@@ -6,5 +6,5 @@
         <link name="front_right_wheel">
             <visual>
-                <origin xyz="0 0 0" rpy="0 0 0"/>
+                <origin xyz="0.2548 -0.03 0.033" rpy="-${pi/2} 0 0"/>
                 <geometry>
                     <mesh scale="0.001 0.001 0.001" filename="package://rona_robot/meshes/front_right_wheel.stl"/>

File: src/rona_robot/robot_description/rear_left_wheel.xacro (robot description, xacro)
@@ -6,5 +6,5 @@
         <link name="rear_left_wheel">
             <visual>
-                <origin xyz="0 0 0" rpy="0 0 0"/>
+                <origin xyz="0.0451 -0.03 -0.1691" rpy="-${pi/2} 0 0"/>
                 <geometry>
                     <mesh scale="0.001 0.001 0.001" filename="package://rona_robot/meshes/rear_left_wheel.stl"/>

File: src/rona_robot/robot_description/rear_right_wheel.xacro (robot description, xacro)
@@ -6,5 +6,5 @@
         <link name="rear_right_wheel">
             <visual>
-                <origin xyz="0 0 0" rpy="0 0 0"/>
+                <origin xyz="0.045 -0.03 0.033" rpy="-${pi/2} 0 0"/>
                 <geometry>
                     <mesh scale="0.001 0.001 0.001" filename="package://rona_robot/meshes/rear_right_wheel.stl"/>

File: src/rona_robot/robot_description/robot_core.xacro (robot description, xacro)
@@ -44,9 +44,9 @@
     <xacro:front_left_wheel/>
     <!-- Front right wheel -->
-    <!-- <xacro:front_right_wheel/> -->
+    <xacro:front_right_wheel/>
     <!-- Rear left wheel -->
-    <!-- <xacro:rear_left_wheel/> -->
+    <xacro:rear_left_wheel/>
     <!-- Rear right wheel -->
-    <!-- <xacro:rear_right_wheel/> -->
+    <xacro:rear_right_wheel/>
     <!-- ROBOT DESCRIPTION END -->
 </robot>
