Commit message: need to keep adjusting the front left wheel

File: src/rona_robot/robot_description/front_left_wheel.xacro (robot description, xacro)
@@ -6,5 +6,5 @@
         <link name="front_left_wheel">
             <visual>
-                <origin xyz="0 0 0" rpy="0 0 0"/>
+                <origin xyz="0.2543 -0.02958 -0.169" rpy="-${pi/2} 0 0"/>
                 <geometry>
                     <mesh scale="0.001 0.001 0.001" filename="package://rona_robot/meshes/front_left_wheel.stl"/>

File: src/rona_robot/robot_description/robot_core.xacro (robot description, xacro)
@@ -44,9 +44,9 @@
     <xacro:front_left_wheel/>
     <!-- Front right wheel -->
-    <xacro:front_right_wheel/>
+    <!-- <xacro:front_right_wheel/> -->
     <!-- Rear left wheel -->
-    <xacro:rear_left_wheel/>
+    <!-- <xacro:rear_left_wheel/> -->
     <!-- Rear right wheel -->
-    <xacro:rear_right_wheel/>
+    <!-- <xacro:rear_right_wheel/> -->
     <!-- ROBOT DESCRIPTION END -->
 </robot>

Commit message: NOW GAZEBO WORKING

File: src/rona_robot/robot_description/front_left_wheel.xacro (robot description, xacro)
@@ -5,4 +5,11 @@
     <xacro:macro name="front_left_wheel">
         <link name="front_left_wheel">
+            <inertial>
+                <origin xyz = "0 0 0"/>
+                <mass value="0.4"/>
+                <inertia ixx="0.000239" ixy="0.0" ixz="0.0"
+                        iyy="0.000239" iyz="0.0"
+                        izz="0.000044" />
+            </inertial>
             <visual>
                 <!-- En rviz el eje X es el rojo, el Y el verde y el Z el azul -->

File: src/rona_robot/robot_description/front_right_wheel.xacro (robot description, xacro)
@@ -5,4 +5,11 @@
     <xacro:macro name="front_right_wheel">
         <link name="front_right_wheel">
+            <inertial>
+                <origin xyz = "0 0 0"/>
+                <mass value="0.4"/>
+                <inertia ixx="0.000239" ixy="0.0" ixz="0.0"
+                        iyy="0.000239" iyz="0.0"
+                        izz="0.000044" />
+            </inertial>
             <visual>
                 <origin xyz="0.2548 -0.03 0.033" rpy="-${pi/2} 0 0"/>

File: src/rona_robot/robot_description/rear_left_wheel.xacro (robot description, xacro)
@@ -5,4 +5,11 @@
     <xacro:macro name="rear_left_wheel">
         <link name="rear_left_wheel">
+            <inertial>
+                <origin xyz = "0 0 0"/>
+                <mass value="0.4"/>
+                <inertia ixx="0.000239" ixy="0.0" ixz="0.0"
+                        iyy="0.000239" iyz="0.0"
+                        izz="0.000044" />
+            </inertial>
             <visual>
                 <origin xyz="0.0451 -0.03 -0.1691" rpy="-${pi/2} 0 0"/>

File: src/rona_robot/robot_description/rear_right_wheel.xacro (robot description, xacro)
@@ -5,4 +5,11 @@
     <xacro:macro name="rear_right_wheel">
         <link name="rear_right_wheel">
+            <inertial>
+                <origin xyz = "0 0 0"/>
+                <mass value="0.4"/>
+                <inertia ixx="0.000239" ixy="0.0" ixz="0.0"
+                        iyy="0.000239" iyz="0.0"
+                        izz="0.000044" />
+            </inertial>
             <visual>
                 <origin xyz="0.045 -0.03 0.033" rpy="-${pi/2} 0 0"/>

File: src/rona_robot/robot_description/robot_core.xacro (robot description, xacro)
@@ -1,12 +1,13 @@
 <?xml version="1.0"?>
-<robot xmlns:xacro="http://www.ros.org/wiki/xacro" name="robot">
+<robot xmlns:xacro="http://www.ros.org/wiki/xacro" name="rona">
     <!-- In this file the basic structure of the omnidirectional robot RONA is described -->
-    <xacro:include filename="inertial_macros.xacro"/>
-    <xacro:include filename="front_left_wheel.xacro"/>
-    <xacro:include filename="front_right_wheel.xacro"/>
-    <xacro:include filename="rear_left_wheel.xacro"/>
-    <xacro:include filename="rear_right_wheel.xacro"/>
-    <xacro:include filename="colors.xacro"/>
-    <xacro:include filename="physical_properties.xacro"/>
+    <xacro:include filename="$(find rona_robot)/robot_description/inertial_macros.xacro"/>
+    <xacro:include filename="$(find rona_robot)/robot_description/front_left_wheel.xacro"/>
+    <xacro:include filename="$(find rona_robot)/robot_description/front_right_wheel.xacro"/>
+    <xacro:include filename="$(find rona_robot)/robot_description/rear_left_wheel.xacro"/>
+    <xacro:include filename="$(find rona_robot)/robot_description/rear_right_wheel.xacro"/>
+    <xacro:include filename="$(find rona_robot)/robot_description/colors.xacro"/>
+    <xacro:include filename="$(find rona_robot)/robot_description/physical_properties.xacro"/>
+    <xacro:include filename="$(find rona_robot)/robot_description/rona_gazebo.xacro"/>
     <!-- ROBOT DESCRIPTION START -->
     <!-- Base link -->
