Commit message: Now gazebo working with complex and simple geometr

File: src/rona_robot/complex_description/macros.xacro (robot description, xacro)
@@ -8,5 +8,5 @@
                 <origin xyz="0 0 0" rpy="0 0 0" />
                 <geometry>
-                    <cylinder radius="0,0082" length="0,045"/>
+                    <cylinder radius="0.0082" length="0.045"/>
                 </geometry>
                 <material name="black"/>
@@ -15,10 +15,14 @@
                 <origin xyz="0 0 0" rpy="0 0 0" />
                 <geometry>
-                    <cylinder radius="0,0082" length="0,045"/>
+                    <cylinder radius="0.0082" length="0.045"/>
                 </geometry>
             </collision>
-            <xacro:inertial_cylinder mass="0.001" length="0.045" radius="0.0082">
-                <origen xyz="0 0 0" rpy="0 0 0"/>
-            </xacro:inertial_cylinder>
+            <inertial>
+                <origin xyz="0 0 0"/>
+                <mass value="0.001" />
+                <inertia ixx="8.72e-8" ixy="0.0" ixz="0.0"
+                        iyy="8.72e-8" iyz="0.0"
+                        izz="6.722e-9" />
+            </inertial>
         </link>
         <joint name="${prefix}_${suffix}_roller_joint" type="continuous">
@@ -28,9 +32,4 @@
                 <origin xyz="${cos(theta)*wheel_radius} ${sin(theta)*wheel_radius} 0" rpy="0 ${roller_orientation} ${(pi/2)+theta}"/>
         </joint>
-        <!-- This block provides the simulator (Gazebo) with information on a few additional
-        physical properties. See http://gazebosim.org/tutorials/?tut=ros_urdf for more-->
-        <gazebo reference="${prefix}_${suffix}_roller">
-            <material>Gazebo/Grey</material>
-        </gazebo>
     </xacro:macro>
     <xacro:macro name="wheel" params="prefix suffix radius length mass offset_x offset_y offset_z wheel_roller_orientation">
@@ -49,5 +48,11 @@
                 </geometry>
             </collision>
-            <!-- <xacro:roller_inertial mass="${mass}"/>     -->
+            <inertial>
+                <origin xyz = "0 0 0"/>
+                <mass value="0.4"/>
+                <inertia ixx="0.000239" ixy="0.0" ixz="0.0"
+                        iyy="0.000239" iyz="0.0"
+                        izz="0.000044" />
+            </inertial>
         </link>
         <joint name="${prefix}_${suffix}_wheel_joint" type="continuous">

File: src/rona_robot/complex_description/robot_core.xacro (robot description, xacro)
@@ -1,4 +1,4 @@
 <?xml version="1.0"?>
-<robot xmlns:xacro="http://www.ros.org/wiki/xacro" >
+<robot xmlns:xacro="http://www.ros.org/wiki/xacro" name="rona">
     <!-- In this file the basic structure of the omnidirectional robot RONA is described -->
     <xacro:include filename="inertial_macros.xacro"/>
@@ -35,15 +35,12 @@
         <origin xyz="0 0 0.022"/>
     </joint>
-    <gazebo reference="chassis">
-        <material>Gazebo/Blue</material>
-    </gazebo>
     <!-- Front left wheel -->
-    <xacro:wheel prefix="front" suffix="left" radius="0,0375" length="0,05" mass="0.4" offset_x="${wheel_offset_x}" offset_y="${wheel_offset_y}" offset_z="${wheel_offset_z}" wheel_roller_orientation="${pi/4}"/>
+    <xacro:wheel prefix="front" suffix="left" radius="0.0375" length="0.05" mass="0.4" offset_x="${wheel_offset_x}" offset_y="${wheel_offset_y}" offset_z="${wheel_offset_z}" wheel_roller_orientation="${pi/4}"/>
     <!-- Front right wheel -->
-    <xacro:wheel prefix="front" suffix="right" radius="0,0375" length="0,05" mass="0.4" offset_x="${wheel_offset_x}" offset_y="${-wheel_offset_y}" offset_z="${wheel_offset_z}" wheel_roller_orientation="${-pi/4}"/>
+    <xacro:wheel prefix="front" suffix="right" radius="0.0375" length="0.05" mass="0.4" offset_x="${wheel_offset_x}" offset_y="${-wheel_offset_y}" offset_z="${wheel_offset_z}" wheel_roller_orientation="${-pi/4}"/>
     <!-- Back left wheel -->
-    <xacro:wheel prefix="back" suffix="left" radius="0,0375" length="0,05" mass="0.4" offset_x="${-wheel_offset_x}" offset_y="${wheel_offset_y}" offset_z="${wheel_offset_z}" wheel_roller_orientation="${-pi/4}"/>
+    <xacro:wheel prefix="back" suffix="left" radius="0.0375" length="0.05" mass="0.4" offset_x="${-wheel_offset_x}" offset_y="${wheel_offset_y}" offset_z="${wheel_offset_z}" wheel_roller_orientation="${-pi/4}"/>
     <!-- Back right wheel -->
-    <xacro:wheel prefix="back" suffix="right" radius="0,0375" length="0,05" mass="0.4" offset_x="${-wheel_offset_x}" offset_y="${-wheel_offset_y}" offset_z="${wheel_offset_z}" wheel_roller_orientation="${pi/4}"/>
+    <xacro:wheel prefix="back" suffix="right" radius="0.0375" length="0.05" mass="0.4" offset_x="${-wheel_offset_x}" offset_y="${-wheel_offset_y}" offset_z="${wheel_offset_z}" wheel_roller_orientation="${pi/4}"/>
     <!-- ROBOT DESCRIPTION END -->
 </robot>
